File: pcb/binaryclock.kicad_pcb (KiCad board)
At the start: 2 copper layers, 150 x 100 mm, 36 parts, among them J1 Barrel_Jack, J2 Screw_Terminal_01x02, J3 LevelShifter_LV, J4 LevelShifter_HV, J5 DS3231, U1 WeMos_D1_mini

Commit message: bla
Parts:
- moved R1 3.81 mm to (78.7, 41.9), turned to 270 degrees
Routing:
- net HV_LED: track 10.8 -> 3.81 mm
- net Net-(D2-Pad4): track 91.9 -> 93.5 mm, vias 1 -> 2
Other:
- outline, holes or cut-outs redrawn
- board text added: "Monate"
- board text added: "Tage"
- board text removed: "Monat"
- board text removed: "Tag"
